Commit message: Editted urdf model to xacro file and corrected inertia matrices
Editted urdf model to xacro file and corrected inertia matrices. The model does not broke but cannot control 2nd rotational joint

File: rsd_description/urdf/prrp2.urdf (robot description, URDF)
Before this commit: robot prrp_robot, 11 links, 10 joints
Links:
- removed link link_add1
- removed link link_add2
- removed link link_add3
- removed link link_add4
Joints:
- removed joint pan_joint2
- removed joint pan_joint3
- removed joint pan_joint4
- removed joint pan_joint5
- joint pan_joint: limit lower=-3.14 upper=3.14 effort=300 velocity=0.1 -> (none)
